Commit message: Atualizações

File: RPi/catkin_ws/src/robot_description/urdf/robot_description.urdf (robot description, URDF)
Before this commit: robot robot_description, 5 links, 4 joints
Links:
- added link laser_frame, mass 0.01; collision cylinder length=0.02 radius=0.02; visual cylinder length=0.02 radius=0.02
- link bl_wheel_link: geometry collision cylinder length=0.02 radius=0.048; visual cylinder length=0.02 radius=0.048
- link br_wheel_link: geometry collision cylinder length=0.02 radius=0.048; visual cylinder length=0.02 radius=0.048
- link fl_wheel_link: geometry collision cylinder length=0.02 radius=0.048; visual cylinder length=0.02 radius=0.048
- link fr_wheel_link: geometry collision cylinder length=0.02 radius=0.048; visual cylinder length=0.02 radius=0.048
Joints:
- added joint laser_joint: type fixed, parent base_link, child laser_frame, origin xyz=0.14 0 0.001 rpy=0 0 0
- joint bl_wheel_joint: type continuous -> fixed
- joint br_wheel_joint: axis 0 -1 0 -> 0 1 0; type continuous -> fixed
- joint fl_wheel_joint: type continuous -> fixed
- joint fr_wheel_joint: axis 0 -1 0 -> 0 1 0; type continuous -> fixed

Commit message: Atualização geral

File: RPi/catkin_ws/src/robot_description/urdf/robot_description.urdf (robot description, URDF)
Before this commit: robot robot_description, 6 links, 5 joints
Links:
- removed link bl_wheel_link
- removed link br_wheel_link
- removed link fl_wheel_link
- removed link fr_wheel_link
- removed link laser_frame
- added link base_footprint; visual box size=0.001 0.001 0.001
- added link camera_link; visual box size=0.04 0.07 0.03
- added link depth_camera_link; visual box size=0.02 0.07 0.014
- added link garra1_link, mass 0.026601; collision mesh filename=package://robot_description/meshes/garra1_link.STL; visual mesh filename=package://robot_description/meshes/garra1_link.STL
- added link garra2_link, mass 0.026601; collision mesh filename=package://robot_description/meshes/garra2_link.STL; visual mesh filename=package://robot_description/meshes/garra2_link.STL
- added link manip_link, mass 0.58414; collision mesh filename=package://robot_description/meshes/manip_link.STL; visual mesh filename=package://robot_description/meshes/manip_link.STL
- added link plat_link, mass 0.68186; collision mesh filename=package://robot_description/meshes/plat_link.STL; visual mesh filename=package://robot_description/meshes/plat_link.STL
- added link sensor_link; visual box size=0.05 0.05 0.05
- link base_link: mass 0.36521 -> 1000
Joints:
- removed joint bl_wheel_joint
- removed joint br_wheel_joint
- removed joint fl_wheel_joint
- removed joint fr_wheel_joint
- removed joint laser_joint
- added joint base_link_joint: type fixed, parent base_footprint, child base_link, origin xyz=0.0 0 0 rpy=0 0 0
- added joint camera_joint: type fixed, parent manip_link, child camera_link, origin xyz=0.33 0 -0.065 rpy=0 1.5708 0
- added joint depth_camera_joint: type fixed, parent base_link, child depth_camera_link, origin xyz=0.083 0 -0.09 rpy=0 0.2 0
- added joint garra1_joint: type prismatic, parent manip_link, child garra1_link, origin xyz=0.28556 0 -0.0662 rpy=3.1416 0 0, axis 0 1 0, limit lower=-0.025 upper=0 effort=100 velocity=0.025
- added joint garra2_joint: type prismatic, parent manip_link, child garra2_link, origin xyz=0.28556 0 -0.0662 rpy=3.1416 0 0, axis 0 1 0, limit lower=0 upper=0.025 effort=100 velocity=0.025
- added joint manip_joint: type prismatic, parent plat_link, child manip_link, origin xyz=0 0 0 rpy=0 0 0, axis 0 0 1, limit lower=0 upper=0.38 effort=300 velocity=0.05
- added joint plat_joint: type revolute, parent base_link, child plat_link, origin xyz=0 0 0 rpy=0 0 0, axis 0 0 1, limit lower=-3.490666 upper=3.490666 effort=300 velocity=1.0472
- added joint sensor_joint: type fixed, parent base_link, child sensor_link, origin xyz=0.1 0 0.2 rpy=0 0 0
